File: hardware/kicad/petb1a.kicad_sch (KiCad schematic)
At the start: 31 parts, among them J1 Socket, J2 USB_C_Receptacle_USB2.0, J3 Socket, SW1 B3U-1000P, SW2 B3U-1000P, U1 ESP32-S3-WROOM-1, U3 XC6220B331MR, U4 USBLC6-2P6

Commit message: update schematics
Parts:
- removed C3: 4u7, symbol Device:C_Polarized_Small
- removed SW2: B3U-1000P, Button_Switch_SMD:SW_SPST_B3U-1000P, symbol Switch:SW_Push
- added SW1: TD-1183SA-1.5H-250, petb1a:KEY-SMD_L3.0-W2.5-LS4.0, symbol Switch:SW_Push
- added TP3: +3V3, TestPoint:TestPoint_Pad_D1.0mm, symbol Connector:TestPoint
- C3: renamed from C4; footprint (none) -> Capacitor_SMD:C_0603_1608Metric; Distributor (none) -> LCSC; Distributor Link (none) -> https://www.lcsc.com/product-detail/Multilayer-Ceramic-Capa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; Distributor Part Number (none) -> C100042; Manufacturer (none) -> YAGEO; Manufacturer Part Number (none) -> CC0603KRX7R9BB103; Part Description Ceramic Capacitors 16V 10nF X7R ±10% -> Ceramic Capacitors 50V 10nF X7R ±10%
- C4: renamed from C5; footprint (none) -> Capacitor_SMD:C_0603_1608Metric; Distributor (none) -> LCSC; Distributor Link (none) -> https://www.lcsc.com/product-detail/Multilayer-Ceramic-Capa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; Distributor Part Number (none) -> C1591; Manufacturer (none) -> Samsung Electro-Mechanics; Manufacturer Part Number (none) -> CL10B104KB8NNNC; Part Description Ceramic Capacitor 16V 100nF X7R ±10% -> Ceramic Capacitor 50V 100nF X7R ±10%
- C5: renamed from C2; footprint (none) -> Capacitor_SMD:C_0603_1608Metric; Distributor (none) -> LCSC; Distributor Link (none) -> https://www.lcsc.com/product-detail/Multilayer-Ceramic-Capa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; Distributor Part Number (none) -> C19702; Manufacturer (none) -> Samsung Electro-Mechanics; Manufacturer Part Number (none) -> CL10A106KP8NNNC; Part Description Ceramic Capacitor 16V 10uF X7R ±10% -> Ceramic Capacitor 10V 10uF X5R ±10%
- C6: footprint (none) -> Capacitor_SMD:C_0603_1608Metric; Distributor (none) -> LCSC; Distributor Link (none) -> https://www.lcsc.com/product-detail/Multilayer-Ceramic-Capa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; Distributor Part Number (none) -> C19702; Manufacturer (none) -> Samsung Electro-Mechanics; Manufacturer Part Number (none) -> CL10A106KP8NNNC; Part Description Ceramic Capacitor 16V 10uF X7R ±10% -> Ceramic Capacitor 10V 10uF X5R ±10%
- D2: Distributor (none) -> LCSC; Distributor Link (none) -> https://www.lcsc.com/product-detail/Schottky-Barrier-Diodes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; Distributor Part Number (none) -> C64885; Manufacturer (none) -> MDD（Microdiode Electronics); Manufacturer Part Number (none) -> B5819W; Part Description 0.05mA@40V 0.58V@1A -> SBD 40V 600mV@1A
- D9: value ESD5651N -> LESD5D5.0CT1G; footprint Capacitor_SMD:C_0402_1005Metric -> Diode_SMD:D_SOD-523; Distributor (none) -> LCSC; Distributor Link https://www.lcsc.com/product-detail/span-style-background-c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 -> https://www.lcsc.com/product-detail/Electrostatic-and-Surge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; Distributor Part Number (none) -> C383211; Manufacturer (none) -> LRC; Manufacturer Part Number (none) -> LESD5D5.0CT1G; Part Description (none) -> ESD 9.4A 18.6V 5.6V Bi-Directional 5V
- F1: value 0.75A -> SMD0805P075TF
- FB1: renamed from FB?; Distributor (none) -> LCSC; Distributor Link (none) -> https://www.lcsc.com/product-detail/Ferrite-Beads_TDK-MMZ16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; Distributor Part Number (none) -> C97120
- J1: renamed from J2; value USB_C_Receptacle_USB2.0 -> TYPEC-304-ACP16; footprint Connector_USB:USB_C_Receptacle_XKB_U262-16XN-4BVC11 -> petb1a:USB-C-SMD_TYPE-C-16P-1; Distributor (none) -> LCSC; Distributor Link (none) -> https://www.lcsc.com/product-detail/USB-Connectors_XUNPU-TY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; Distributor Part Number (none) -> C2982555; Manufacturer (none) -> XUNPU; Manufacturer Part Number (none) -> TYPEC-304-ACP16; Part Description (none) -> Type-C SMD 3A 1 Surface Mount，Right Angle 16P Female
- J2: renamed from J1; value Socket -> DNP; footprint (none) -> Connector_PinSocket_2.54mm:PinSocket_1x22_P2.54mm_Vertical; Part Description (none) -> Pin Header 1x22 P2.54mm Vertical
- J3: value Socket -> DNP; footprint (none) -> Connector_PinSocket_2.54mm:PinSocket_1x22_P2.54mm_Vertical; Part Description (none) -> Pin Header 1x22 P2.54mm Vertical
- JP1: footprint (none) -> Jumper:SolderJumper-2_P1.3mm_Open_RoundedPad1.0x1.5mm
- SW2: renamed from SW1; value B3U-1000P -> TD-1183SA-1.5H-250; footprint Button_Switch_SMD:SW_SPST_B3U-1000P -> petb1a:KEY-SMD_L3.0-W2.5-LS4.0; Distributor (none) -> LCSC; Distributor Link (none) -> https://www.lcsc.com/product-detail/Tactile-Switches_DEALON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; Distributor Part Number (none) -> C2905189; Manufacturer (none) -> DEALON; Manufacturer Part Number (none) -> TD-1183SA-1.5H-250; Part Description (none) -> Tactile Switches 2.5mm 1.5mm 3mm SMD,2.5x3mm
- U3: value XC6220B331MR -> XC6220B331MR-G; Distributor (none) -> LCSC; Distributor Link (none) -> https://www.lcsc.com/product-detail/Linear-Voltage-Regulato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; Distributor Part Number (none) -> C86534; Manufacturer (none) -> Torex Semicon; Manufacturer Part Number (none) -> XC6220B331MR-G; Part Description (none) -> LDO 50dB@(1kHz) 1A Fixed 3.3V Positive
- renumbered C7 to C1, C8 to C2, C1 to C7, C9 to C8, R5 to R4, R6 to R5, R4 to R6, U4 to U1, U1 to U2
Connections:
- net LED0 is gone; now on net GPIO38: JP1.1 (A)
- net +3V3: now also TP3.1
- net BOOT0: now also J3.14 (Pin_14), SW1.2
- net GND: now also J3.1 (Pin_1), J3.21 (Pin_21), J3.22 (Pin_22), SW1.1
- net GPIO1: now also J3.4 (Pin_4)
- net GPIO2: now also J3.5 (Pin_5)
- net GPIO21: now also J3.18 (Pin_18)
- net GPIO35: now also J3.13 (Pin_13)
- net GPIO36: now also J3.12 (Pin_12)
- net GPIO37: now also J3.11 (Pin_11)
- net GPIO38: now also J3.10 (Pin_10)
- net GPIO39: now also J3.9 (Pin_9)
- net GPIO40: now also J3.8 (Pin_8)
- net GPIO41: now also J3.7 (Pin_7)
- net GPIO42: now also J3.6 (Pin_6)
- net GPIO45: now also J3.15 (Pin_15)
- net GPIO47: now also J3.17 (Pin_17)
- net GPIO48: now also J3.16 (Pin_16)
- net U0RXD: now also J3.3 (Pin_3)
- net U0TXD: now also J3.2 (Pin_2)
- net GPIO20: now reaches J3.19 (Pin_19)
- net GPIO19: now reaches J3.20 (Pin_20)
Other:
- note added: "750mA"
- note added: "Breakout Socket"
- note added: "ESP32-S3 Module"
- note added: "Max Power Output : 1 A Quiescent Current : 8 uA in HS Mode 50 uA in PS Mode"
- note added: "See ESP32-S3 Hardware Design Guidelines Chapter 3.2"
- note removed: "Max 1A"
- note removed: "Place Cap Close to Chip"
- note removed: "See ESP32-C6 Hardware Design Guidelines Chapter 2.2"
- title: PETB1A -> Teapotlabs PETB1A
- moved on the sheet: C1, C2, C3, C4, C7, C8, D3, F1, FB1, J2, J3, JP1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

Commit message: change socket to header
Parts:
- J2, J3: footprint Connector_PinSocket_2.54mm:PinSocket_1x22_P2.54mm_Vertical -> Connector_PinHeader_2.54mm:PinHeader_1x22_P2.54mm_Vertical
Changed lines of the file:
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@@
       (effects (font (size 1.27 1.27)) (justify left))
     )
-    (property "Footprint" "Connector_PinSocket_2.54mm:PinSocket_1x22_P2.54mm_Vertical" (at 194.31 107.95 0)
+    (property "Footprint" "Connector_PinHeader_2.54mm:PinHeader_1x22_P2.54mm_Vertical" (at 194.31 107.95 0)
       (effects (font (size 1.27 1.27)) hide)
     )
@@
       (effects (font (size 1.27 1.27)) (justify left))
     )
-    (property "Footprint" "Connector_PinSocket_2.54mm:PinSocket_1x22_P2.54mm_Vertical" (at 181.61 107.95 0)
-      (effects (font (size 1.27 1.27)) hide)
-    )
+    (property "Footprint" "Connector_PinHeader_2.54mm:PinHeader_1x22_P2.54mm_Vertical" (at 181.61 107.95 0)
+      (effects (font (size 1.27 1.27)) hide)
+    )

Commit message: intial pcb wiring
Parts:
- removed U2: ESP32-S3-WROOM-1, Espressif:ESP32-S3-WROOM-1, symbol Espressif:ESP32-S3-WROOM-1
- added U2: ESP32-S3-WROOM-1, petb1a:ESP32-S3-WROOM-1, symbol petb1a:ESP32-S3-WROOM-1
- C1: footprint (none) -> Capacitor_SMD:C_0603_1608Metric; Distributor (none) -> LCSC; Distributor Link (none) -> https://www.lcsc.com/product-detail/Multilayer-Ceramic-Capa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; Distributor Part Number (none) -> C19702; Manufacturer (none) -> Samsung Electro-Mechanics; Manufacturer Part Number (none) -> CL10A106KP8NNNC; Part Description Ceramic Capacitors 16V 10nF X7R ±10% -> Ceramic Capacitor 10V 10uF X5R ±10%
- C2: footprint (none) -> Capacitor_SMD:C_0603_1608Metric; Distributor (none) -> LCSC; Distributor Link (none) -> https://www.lcsc.com/product-detail/Multilayer-Ceramic-Capa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; Distributor Part Number (none) -> C1591; Manufacturer (none) -> Samsung Electro-Mechanics; Manufacturer Part Number (none) -> CL10B104KB8NNNC; Part Description Ceramic Capacitor 16V 100nF X7R ±10% -> Ceramic Capacitor 50V 100nF X7R ±10%
Connections:
- net +3V3: now also U2.2 (3V3)
- net BOOT0: now also U2.27 (GPIO0/BOOT)
- net CHIP_EN: now also U2.3 (EN)
- net D_OUT+: now also U2.14 (GPIO20/U1CTS/ADC2_CH9/CLK_OUT1/USB_D+)
- net D_OUT-: now also U2.13 (GPIO19/U1RTS/ADC2_CH8/CLK_OUT2/USB_D-)
- net GND: now also U2.1 (GND), U2.40 (GND), U2.41 (GND)
- net GPIO1: now also U2.39 (GPIO1/TOUCH1/ADC1_CH0)
- net GPIO10: now also U2.18 (GPIO10/TOUCH10/ADC1_CH9/FSPICS0/FSPIIO4/SUBSPICS0)
- net GPIO11: now also U2.19 (GPIO11/TOUCH11/ADC2_CH0/FSPID/FSPIIO5/SUBSPID)
- net GPIO12: now also U2.20 (GPIO12/TOUCH12/ADC2_CH1/FSPICLK/FSPIIO6/SUBSPICLK)
- net GPIO13: now also U2.21 (GPIO13/TOUCH13/ADC2_CH2/FSPIQ/FSPIIO7/SUBSPIQ)
- net GPIO14: now also U2.22 (GPIO14/TOUCH14/ADC2_CH3/FSPIWP/FSPIDQS/SUBSPIWP)
- net GPIO15: now also U2.8 (GPIO15/U0RTS/ADC2_CH4/XTAL_32K_P)
- net GPIO16: now also U2.9 (GPIO16/U0CTS/ADC2_CH5/XTAL_32K_N)
- net GPIO17: now also U2.10 (GPIO17/U1TXD/ADC2_CH6)
- net GPIO18: now also U2.11 (GPIO18/U1RXD/ADC2_CH7/CLK_OUT3)
- net GPIO2: now also U2.38 (GPIO2/TOUCH2/ADC1_CH1)
- net GPIO21: now also U2.23 (GPIO21)
- net GPIO3: now also U2.15 (GPIO3/TOUCH3/ADC1_CH2)
- net GPIO35: now also U2.28 (SPIIO6/GPIO35/FSPID/SUBSPID)
- net GPIO36: now also U2.29 (SPIIO7/GPIO36/FSPICLK/SUBSPICLK)
- net GPIO37: now also U2.30 (SPIDQS/GPIO37/FSPIQ/SUBSPIQ)
- net GPIO38: now also U2.31 (GPIO38/FSPIWP/SUBSPIWP)
- net GPIO39: now also U2.32 (MTCK/GPIO39/CLK_OUT3/SUBSPICS1)
- net GPIO4: now also U2.4 (GPIO4/TOUCH4/ADC1_CH3)
- net GPIO40: now also U2.33 (MTDO/GPIO40/CLK_OUT2)
- net GPIO41: now also U2.34 (MTDI/GPIO41/CLK_OUT1)
- net GPIO42: now also U2.35 (MTMS/GPIO42)
- net GPIO45: now also U2.26 (GPIO45)
- net GPIO46: now also U2.16 (GPIO46)
- net GPIO47: now also U2.24 (GPIO47/SPICLK_P/SUBSPICLK_P_DIFF)
- net GPIO48: now also U2.25 (GPIO48/SPICLK_N/SUBSPICLK_N_DIFF)
- net GPIO5: now also U2.5 (GPIO5/TOUCH5/ADC1_CH4)
- net GPIO6: now also U2.6 (GPIO6/TOUCH6/ADC1_CH5)
- net GPIO7: now also U2.7 (GPIO7/TOUCH7/ADC1_CH6)
- net GPIO8: now also U2.12 (GPIO8/TOUCH8/ADC1_CH7/SUBSPICS1)
- net GPIO9: now also U2.17 (GPIO9/TOUCH9/ADC1_CH8/FSPIHD/SUBSPIHD)
- net U0RXD: now also U2.36 (U0RXD/GPIO44/CLK_OUT2)
- net U0TXD: now also U2.37 (U0TXD/GPIO43/CLK_OUT1)
Other:
- note added: "Header should be 2.54mm pitch for a breadboard friendly development board"
- note added: "Length between header should be atlest 2.54mm*3 to fit in breadboard"
- moved on the sheet: J2, J3

Commit message: update pcb layout
Connections:
- net +3V3: now also D3.2 (A); no longer R6.1
- net at R6.2: now also JP1.2 (B); no longer D3.2 (A)
- net at D3.1 (K): now also R6.1; no longer JP1.2 (B)
Other:
- moved on the sheet: D3, R6
Changed lines of the file:
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@@
     (stroke (width 0) (type default))
   )
-  (wire (pts (xy 260.35 139.7) (xy 262.89 139.7))
+  (wire (pts (xy 257.81 139.7) (xy 260.35 139.7))
     (stroke (width 0) (type default))
   )
@@
     )
   )
-  (symbol (lib_id "Device:R_Small") (at 265.43 139.7 270) (mirror x) (unit 1)
-    (in_bom yes) (on_board yes) (dnp no)
-    (property "Reference" "R6" (at 263.525 142.24 90)
-      (effects (font (size 1.27 1.27)))
-    )
-    (property "Value" "1K" (at 267.335 142.24 90)
-      (effects (font (size 1.27 1.27)))
-    )
-    (property "Footprint" "Resistor_SMD:R_0603_1608Metric" (at 265.43 139.7 0)
-      (effects (font (size 1.27 1.27)) hide)
-    )
-    (property "Datasheet" "~" (at 265.43 139.7 0)
+  (symbol (lib_id "Device:R_Small") (at 255.27 139.7 270) (mirror x) (unit 1)
+    (in_bom yes) (on_board yes) (dnp no)
+    (property "Reference" "R6" (at 253.365 142.24 90)
+      (effects (font (size 1.27 1.27)))
+    )
+    (property "Value" "1K" (at 257.175 142.24 90)
+      (effects (font (size 1.27 1.27)))
+    )
+    (property "Footprint" "Resistor_SMD:R_0603_1608Metric" (at 255.27 139.7 0)
+      (effects (font (size 1.27 1.27)) hide)
+    )
+    (property "Datasheet" "~" (at 255.27 139.7 0)
       (effects (font (size 1.27 1.27)) hide)
     )
@@
     )
   )
-  (symbol (lib_id "Device:LED") (at 256.54 139.7 0) (mirror x) (unit 1)
-    (in_bom yes) (on_board yes) (dnp no)
-    (property "Reference" "D3" (at 254.635 135.89 0)
-      (effects (font (size 1.27 1.27)))
-    )
-    (property "Value" "RED" (at 259.08 135.89 0)
-      (effects (font (size 1.27 1.27)))
-    )
-    (property "Footprint" "LED_SMD:LED_0603_1608Metric" (at 256.54 139.7 0)
-      (effects (font (size 1.27 1.27)) hide)
-    )
-    (property "Datasheet" "~" (at 256.54 139.7 0)
-      (effects (font (size 1.27 1.27)) hide)
-    )
-    (property "Part Description" "" (at 256.54 139.7 0)
-      (effects (font (size 1.27 1.27)) hide)
-    )
-    (property "Manufacturer" "" (at 256.54 139.7 0)
-      (effects (font (size 1.27 1.27)) hide)
-    )
-    (property "Manufacturer Part Number" "" (at 256.54 139.7 0)
-      (effects (font (size 1.27 1.27)) hide)
-    )
-    (property "Distributor" "" (at 256.54 139.7 0)
-      (effects (font (size 1.27 1.27)) hide)
-    )
-    (property "Distributor Part Number" "" (at 256.54 139.7 0)
-      (effects (font (size 1.27 1.27)) hide)
-    )
-    (property "Distributor Link" "" (at 256.54 139.7 0)
-      (effects (font (size 1.27 1.27)) hide)
-    )
+  (symbol (lib_id "Device:LED") (at 264.16 139.7 0) (mirror x) (unit 1)
+    (in_bom yes) (on_board yes) (dnp no)
+    (property "Reference" "D3" (at 262.255 135.89 0)
+      (effects (font (size 1.27 1.27)))
+    )
+    (property "Value" "RED" (at 266.7 135.89 0)
+      (effects (font (size 1.27 1.27)))
+    )
+    (property "Footprint" "LED_SMD:LED_0603_1608Metric" (at 264.16 139.7 0)
+      (effects (font (size 1.27 1.27)) hide)
+    )
+    (property "Datasheet" "~" (at 264.16 139.7 0)
+      (effects (font (size 1.27 1.27)) hide)
+    )
+    (property "Part Description" "" (at 264.16 139.7 0)
+      (effects (font (size 1.27 1.27)) hide)
+    )
+    (property "Manufacturer" "" (at 264.16 139.7 0)
+      (effects (font (size 1.27 1.27)) hide)
+    )
+    (property "Manufacturer Part Number" "" (at 264.16 139.7 0)
+      (effects (font (size 1.27 1.27)) hide)
+    )
+    (property "Distributor" "" (at 264.16 139.7 0)
+      (effects (font (size 1.27 1.27)) hide)
+    )
+    (property "Distributor Part Number" "" (at 264.16 139.7 0)
+      (effects (font (size 1.27 1.27)) hide)
+    )
+    (property "Distributor Link" "" (at 264.16 139.7 0)
+      (effects (font (size 1.27 1.27)) hide)
+    )

Commit message: update pcb
Parts:
- J2, J3: footprint Connector_PinHeader_2.54mm:PinHeader_1x22_P2.54mm_Vertical -> petb1a:PinHeader_1x22_P2.54mm_Vertical
Changed lines of the file:
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@@
       (effects (font (size 1.27 1.27)) (justify left))
     )
-    (property "Footprint" "Connector_PinHeader_2.54mm:PinHeader_1x22_P2.54mm_Vertical" (at 194.31 112.395 0)
+    (property "Footprint" "petb1a:PinHeader_1x22_P2.54mm_Vertical" (at 194.31 112.395 0)
       (effects (font (size 1.27 1.27)) hide)
     )
@@
       (effects (font (size 1.27 1.27)) (justify left))
     )
-    (property "Footprint" "Connector_PinHeader_2.54mm:PinHeader_1x22_P2.54mm_Vertical" (at 181.61 112.395 0)
-      (effects (font (size 1.27 1.27)) hide)
-    )
+    (property "Footprint" "petb1a:PinHeader_1x22_P2.54mm_Vertical" (at 181.61 112.395 0)
+      (effects (font (size 1.27 1.27)) hide)
+    )

Commit message: update board
Parts:
- removed J2, J3: DNP, petb1a:PinHeader_1x22_P2.54mm_Vertical, symbol Connector_Generic:Conn_01x22
- removed JP1: EN_LED0, Jumper:SolderJumper-2_P1.3mm_Open_RoundedPad1.0x1.5mm, symbol Jumper:SolderJumper_2_Open
- added C10, C9: 100n, Capacitor_SMD:C_0402_1005Metric, symbol Device:C_Small
- added D4: GREEN, LED_SMD:LED_0603_1608Metric, symbol Device:LED
- added H1, H2, H3, H4: MountingHole, MountingHole:MountingHole_3.2mm_M3, symbol Mechanical:MountingHole
- added J2: EXP1, petb1a:JST_SH_SM04B-SRSS-TB_1x04-1MP_P1.00mm_Horizontal, symbol Connector_Generic:Conn_01x04
- added J3: EXP2, petb1a:JST_SH_SM04B-SRSS-TB_1x04-1MP_P1.00mm_Horizontal, symbol Connector_Generic:Conn_01x04
- added J4: Qwiic, petb1a:JST_SH_SM04B-SRSS-TB_1x04-1MP_P1.00mm_Horizontal, symbol Connector_Generic:Conn_01x04
- added R10, R11, R12, R13, R8, R9: 10K, Resistor_SMD:R_0402_1005Metric, symbol Device:R_Small
- added R7: 1K, Resistor_SMD:R_0603_1608Metric, symbol Device:R_Small
- added U4: BME680, petb1a:Bosch_LGA-8_3x3mm_P0.8mm_ClockwisePinNumbering, symbol Sensor:BME680
- TP1: value VBUS_IN -> VBUSIN
Connections:
- net GPIO18 is gone; now on net LED0: U2.11 (GPIO18/U1RXD/ADC2_CH7/CLK_OUT3)
- net +3V3: now also C10.2, C9.1, D4.2 (A), J4.2 (Pin_2), R10.1, R11.2, R12.1, R13.2, R8.2, R9.2, U4.6 (VDDIO), U4.8 (VDD)
- net GND: now also C10.1, C9.2, J4.1 (Pin_1), U4.1 (GND), U4.7 (GND)
- net GPIO1: now also J2.1 (Pin_1)
- net GPIO11: now also J4.3 (Pin_3), R12.2
- net GPIO12: now also J4.4 (Pin_4), R13.1
- net GPIO2: now also J2.2 (Pin_2)
- net GPIO3: now also J3.4 (Pin_4)
- net GPIO36: now also R10.2, U4.3 (SDI)
- net GPIO37: now also R11.1, U4.4 (SCK)
- net GPIO4: now also J3.3 (Pin_3)
- net GPIO5: now also J3.2 (Pin_2)
- net GPIO6: now also J3.1 (Pin_1)
- net U0RXD: now also J2.4 (Pin_4)
- net U0TXD: now also J2.3 (Pin_3)
- net LED0: now reaches R6.2
- net GPIO10: no longer names the net of U2.18 (GPIO10/TOUCH10/ADC1_CH9/FSPICS0/FSPIIO4/SUBSPICS0)
- net GPIO13: no longer names the net of U2.21 (GPIO13/TOUCH13/ADC2_CH2/FSPIQ/FSPIIO7/SUBSPIQ)
- net GPIO14: no longer names the net of U2.22 (GPIO14/TOUCH14/ADC2_CH3/FSPIWP/FSPIDQS/SUBSPIWP)
- net GPIO15: no longer names the net of U2.8 (GPIO15/U0RTS/ADC2_CH4/XTAL_32K_P)
- net GPIO16: no longer names the net of U2.9 (GPIO16/U0CTS/ADC2_CH5/XTAL_32K_N)
- net GPIO17: no longer names the net of U2.10 (GPIO17/U1TXD/ADC2_CH6)
- net GPIO21: no longer names the net of U2.23 (GPIO21)
- net GPIO35: no longer names the net of U2.28 (SPIIO6/GPIO35/FSPID/SUBSPID)
- net GPIO38: no longer names the net of U2.31 (GPIO38/FSPIWP/SUBSPIWP)
- net GPIO39: no longer names the net of U2.32 (MTCK/GPIO39/CLK_OUT3/SUBSPICS1)
- net GPIO40: no longer names the net of U2.33 (MTDO/GPIO40/CLK_OUT2)
- net GPIO41: no longer names the net of U2.34 (MTDI/GPIO41/CLK_OUT1)
- net GPIO42: no longer names the net of U2.35 (MTMS/GPIO42)
- net GPIO45: no longer names the net of U2.26 (GPIO45)
- net GPIO46: no longer names the net of U2.16 (GPIO46)
- net GPIO47: no longer names the net of U2.24 (GPIO47/SPICLK_P/SUBSPICLK_P_DIFF)
- net GPIO48: no longer names the net of U2.25 (GPIO48/SPICLK_N/SUBSPICLK_N_DIFF)
- net GPIO7: no longer names the net of U2.7 (GPIO7/TOUCH7/ADC1_CH6)
- net GPIO8 renamed LED1
- net LED1: now also R7.2
- net GPIO9: no longer names the net of U2.17 (GPIO9/TOUCH9/ADC1_CH8/FSPIHD/SUBSPIHD)
- new net: R8.1, U4.5 (SDO)
- new net: D4.1 (K), R7.1
- new net: R9.1, U4.2 (CSB)
- no-connect marks 3 -> 22
Other:
- note added: "90Ohm Differential Impedance Trace for USB"
- note added: "Environmental Sensor"
- note added: "Expansion Connector"
- note added: "I2C Address: 0x77"
- note added: "I2C Pull-up"
- note removed: "Breakout Socket"
- note removed: "Header should be 2.54mm pitch for a breadboard friendly development board"
- note removed: "Length between header should be atlest 2.54mm*3 to fit in breadboard"
- note removed: "USB trace is less than Critical Length (2.4 inch) for USB2.0 Full-speed specification. Impedance control is not crucial."
- moved on the sheet: C1, C2, C3, C4, C5, C6, C7, C8, D2, D3, D9, F1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
