File: hardware/kicad/petb1a.kicad_sch (KiCad schematic)
At the start: 46 parts, among them J1 TYPEC-304-ACP16, J2 EXP1, J3 EXP2, J4 Qwiic, SW1 TD-1183SA-1.5H-250, SW2 TD-1183SA-1.5H-250, U1 USBLC6-2P6, U2 ESP32-S3-WROOM-1, U3 XC6220B331MR-G, U4 BME680

Commit message: revision 1 design
Parts:
- removed D2: B5819W, Diode_SMD:D_SOD-123, symbol Diode:MBR0540
- C1, C5, C6: Part Description Ceramic Capacitor 10V 10uF X5R ±10% -> (none)
- C10, C9: Distributor (none) -> LCSC; Distributor Link (none) -> https://www.lcsc.com/product-detail/Multilayer-Ceramic-Capa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; Distributor Part Number (none) -> C77020; Manufacturer (none) -> Murata Electronics; Manufacturer Part Number (none) -> GRM155R71H104KE14D
- C2, C4: Part Description Ceramic Capacitor 50V 100nF X7R ±10% -> (none)
- C3: Part Description Ceramic Capacitors 50V 10nF X7R ±10% -> (none)
- C7, C8: Part Description Ceramic Capacitors 10V 1uF X7R ±10% -> (none)
- D3: value RED -> XL-1608SURC-06; Distributor (none) -> LCSC; Distributor Link (none) -> https://www.lcsc.com/product-detail/Light-Emitting-Diodes-s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; Distributor Part Number (none) -> C965799; Manufacturer (none) -> XINGLIGHT; Manufacturer Part Number (none) -> XL-1608SURC-06
- D4: value GREEN -> NCD0603C4; Distributor (none) -> LCSC; Distributor Link (none) -> https://www.lcsc.com/product-detail/Light-Emitting-Diodes-s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; Distributor Part Number (none) -> C7429911; Manufacturer (none) -> Foshan NationStar Optoelectronics; Manufacturer Part Number (none) -> NCD0603C4
- D9: Part Description ESD 9.4A 18.6V 5.6V Bi-Directional 5V -> (none)
- F1: Part Description Resettable Fuses 6V 750mA 40A 1.5A -> (none)
- FB1: Part Description Ferrite Beads 400mΩ ±25% 600Ω@100MHz -> (none)
- J1: Part Description Type-C SMD 3A 1 Surface Mount，Right Angle 16P Female -> (none)
- J2: value EXP1 -> SM04B-SRSS-TB(LF)(SN); Distributor (none) -> LCSC; Distributor Link (none) -> https://www.lcsc.com/product-detail/Wire-To-Board-Wire-To-W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; Distributor Part Number (none) -> C160404; Manufacturer JST Sales America -> JST; Manufacturer Part Number (none) -> SM04B-SRSS-TB(LF)(SN); Part Number SM04B-SRSS-TB -> (none)
- J3: value EXP2 -> SM04B-SRSS-TB(LF)(SN); Distributor (none) -> LCSC; Distributor Link (none) -> https://www.lcsc.com/product-detail/Wire-To-Board-Wire-To-W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; Distributor Part Number (none) -> C160404; Manufacturer JST Sales America -> JST; Manufacturer Part Number (none) -> SM04B-SRSS-TB(LF)(SN); Part Number SM04B-SRSS-TB -> (none)
- J4: value Qwiic -> SM04B-SRSS-TB(LF)(SN); Distributor (none) -> LCSC; Distributor Link (none) -> https://www.lcsc.com/product-detail/Wire-To-Board-Wire-To-W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; Distributor Part Number (none) -> C160404; Manufacturer JST Sales America -> JST; Manufacturer Part Number (none) -> SM04B-SRSS-TB(LF)(SN); Part Number SM04B-SRSS-TB -> (none)
- R1, R2, R3: Part Description Resistor 62.5mW ±1% 5.1kΩ -> (none)
- R10, R11, R12, R13, R4, R5, R8, R9: Part Description Resistors 62.5mW ±1% 10kΩ -> (none)
- R6, R7: Distributor (none) -> LCSC; Distributor Link (none) -> https://www.lcsc.com/product-detail/Chip-Resistor-Surface-M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; Distributor Part Number (none) -> C22548; Manufacturer (none) -> YAGEO; Manufacturer Part Number (none) -> RC0603FR-071KL
- SW1, SW2: Part Description Tactile Switches 2.5mm 1.5mm 3mm SMD,2.5x3mm -> (none)
- U1: Part Description ESD Protection 6V 17V 2 Unidirectional 5.25V -> (none)
- U2: Distributor (none) -> LCSC; Distributor Link (none) -> https://www.lcsc.com/product-detail/WiFi-Modules_Espressif-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; Distributor Part Number (none) -> C2913202; Manufacturer (none) -> Espressif Systems; Manufacturer Part Number (none) -> ESP32-S3-WROOM-1-N16R8
- U3: Part Description LDO 50dB@(1kHz) 1A Fixed 3.3V Positive -> (none)
- U4: Distributor (none) -> LCSC; Distributor Link (none) -> https://www.lcsc.com/product-detail/Temperature-and-Humidit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; Distributor Part Number (none) -> C3664478; Manufacturer (none) -> Bosch Sensortec; Manufacturer Part Number (none) -> BME688
Connections:
- net +5V is gone; now on net VBUS: C5.1, R3.1, U3.1 (VIN)
Other:
- note added: "GREEN"
- note added: "RED"
- moved on the sheet: C5, C6, J4, R3, TP3, U3
